File: PCBs/Button_PCB/Button_PCB.kicad_sch (KiCad schematic)
At the start: 4 parts, among them J1 Conn_01x05_Male, J2 RIGHT_BUTTON, J3 MIDDLE_BUTTON, J4 LEFT_BUTTON

Commit message: V3.4.3-alpha Generated PCB Gerber Files
Connections:
- net GND: now reaches J1.2 (Pin_2), J2.1 (Pin_1), J3.1 (Pin_1), J4.1 (Pin_1)
- net VCC: now reaches J1.1 (Pin_1), J2.3 (Pin_3), J3.3 (Pin_3), J4.3 (Pin_3)
