File: PCBs/Light_PCB/Light_PCB.kicad_pcb (KiCad board)
At the start: 2 copper layers, 70 x 70 mm, 19 parts, among them J1 Conn_01x03_Male, Q1 2N3904

Commit message: V3.4.1-alpha Added PCB Labels
Other:
- board text added: "GND"
- board text added: "IN"
- board text added: "Sunrise Alarm V3: Light PCB V1"
- board text added: "VCC"
Changed lines of the file:
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@@
   (gr_line (start 160 63) (end 160 107) (layer "User.4") (width 0.1))
   (gr_line (start 110 107) (end 110 63) (layer "User.4") (width 0.1))
+  (gr_text "GND" (at 134.99 66.39) (layer "B.SilkS")
+    (effects (font (size 1.5 0.8) (thickness 0.15)) (justify mirror))
+  )
+  (gr_text "Sunrise Alarm V3: Light PCB V1" (at 135 83.98) (layer "B.SilkS")
+    (effects (font (size 1.5 1.5) (thickness 0.15)) (justify mirror))
+  )
+  (gr_text "VCC" (at 137.53 66.4) (layer "B.SilkS")
+    (effects (font (size 1.5 0.8) (thickness 0.15)) (justify mirror))
+  )
+  (gr_text "IN" (at 132.43 66.38) (layer "B.SilkS")
+    (effects (font (size 1.5 0.8) (thickness 0.15)) (justify mirror))
+  )
   (dimension (type aligned) (layer "Dwgs.User")
     (pts (xy 164.5 70.85) (xy 164.5 85))
